File: Mic Schematic/Mic Schematic.kicad_sch (KiCad schematic)
At the start: 38 parts, among them J1 Conn_01x03, SW1 SW_DPDT_x2, U2 NE5532, U3 NE5532

Commit message: Completed
Parts:
- removed C10: 150pF, symbol Device:C
- removed C4, C7, C8: 2.2uF, symbol Device:C_Polarized
- removed C9: 33uF, symbol Device:C_Polarized
- removed J1: Conn_01x03, symbol Connector_Generic:Conn_01x03
- removed R10, R11, R16: 1k, symbol Device:R
- removed R12: 680, symbol Device:R
- removed R14: 10k, symbol Device:R
- removed R17: 5.1K, symbol Device:R
- removed R8, R9: 2.2k, symbol Device:R
- removed RV2: 10k, symbol Device:R_Potentiometer
- removed Right_1, Right_2: Conn_01x02, symbol Connector_Generic:Conn_01x02
- removed SW1: SW_DPDT_x2, symbol Switch:SW_DPDT_x2
- removed U1: (no value), symbol custom_component:NE5532
- removed U3: NE5532, PCM_JLCPCB:SOIC-8_L4.9-W3.9-P1.27-LS6.0-BL, symbol Amplifier_Operational:NE5532
- added C12: 2.2uF, symbol Device:C_Polarized
- added C7: 120pF, symbol Device:C
- added Left_Output: Conn_01x02, symbol Connector_Generic:Conn_01x02
- added R13, R18: 100k, symbol Device:R
- R1, R5: value 2.2k -> 6.8k
- U2: value NE5532 -> NE5532/OP2134
Connections:
- net +9V: now also C11.2, C12.1, C7.2
- net GND: now also C11.1, C12.2, C7.1, Left_Output.2 (Pin_2), R13.2, R18.1
- net at C1.1, R7.1: now also R18.2
- net at C2.2, RV1.2, U2.1: now also R15.2, R4.2
- net at R15.1: now also Left_Output.1 (Pin_1)
- net at C5.1, R6.1: now also R13.1
- no-connect marks 2 -> 1
Other:
- note added: "Add decoupling capacitor to V+ and V-"
- moved on the sheet: C6, Left_1, Left_2, R15, R4, R6, R7
