File: Mic Schematic/untitled.kicad_sch (KiCad schematic)
At the start: 23 parts, among them U2 NE5532/OP2134

Commit message: Update schematic
Parts:
- removed C1, C11, C12, C5: 2.2uF, symbol Device:C_Polarized
- removed C2: 150pF, symbol Device:C
- removed C3: 33uF, symbol Device:C_Polarized
- removed C6, C7: 120pF, symbol Device:C
- removed Left_1, Left_2, Left_Output: Conn_01x02, symbol Connector_Generic:Conn_01x02
- removed R1, R5: 6.8k, symbol Device:R
- removed R13, R18: 100k, symbol Device:R
- removed R15, R6, R7: 1k, symbol Device:R
- removed R2: 5.1K, symbol Device:R
- removed R3: 680, symbol Device:R
- removed R4: 10k, symbol Device:R
- removed RV1: 50K, symbol Device:R_Potentiometer
- removed U2: NE5532/OP2134, PCM_JLCPCB:SOIC-8_L4.9-W3.9-P1.27-LS6.0-BL, symbol Amplifier_Operational:NE5532
- added C10: 150pF, symbol Device:C
- added C13, C14: 2.2uF, symbol Device:C_Polarized
- added C15, C16: 120pF, symbol Device:C
- added C8: 22nF -> 10nF, symbol Device:C
- added C9: 33uF, symbol Device:C_Polarized
- added Left_3, Left_Output1: Conn_01x02, symbol Connector_Generic:Conn_01x02
- added R10, R20: 1k, symbol Device:R
- added R12: 680, symbol Device:R
- added R14: 100k, symbol Device:R
- added R16: 5.1K, symbol Device:R
- added R17: 10k, symbol Device:R
- added R8: 6.8k, symbol Device:R
- added RV2: 50K, symbol Device:R_Potentiometer
- added U3: NE5532/OP2134, PCM_JLCPCB:SOIC-8_L4.9-W3.9-P1.27-LS6.0-BL, symbol Amplifier_Operational:NE5532
Connections:
- net +9V: now also C13.1, C15.2, R8.1
- net -9V: now also C14.2, C16.1
- net GND: now also C13.2, C14.1, C15.1, C16.2, C9.2, Left_3.1 (Pin_1), Left_Output1.2 (Pin_2), R14.2, R17.1
- new net: C8.2, R10.1, R14.1
- new net: R10.2, U3.3 (+)
- new net: C10.2, R17.2, R20.2, RV2.2, U3.1
- new net: R16.2, RV2.3
- new net: C9.1, R12.1
- new net: C10.1, R12.2, R16.1, U3.2 (-)
- new net: Left_Output1.1 (Pin_1), R20.1
- new net: C8.1, Left_3.2 (Pin_2), R8.2
Other:
- removed sheet mini shit
- note added: "C8 Low-freq / bass cutoff Increase -> More bass Decrease -> Remove more bass C10 High-freq / treble cutoff Increase -> Remove high pitch Decrease -> Allow more high pitch"

Commit message: Update schematic
Parts:
- removed C13, C14: 2.2uF, symbol Device:C_Polarized
- removed C15, C16: 120pF, symbol Device:C
- removed U3: NE5532/OP2134, PCM_JLCPCB:SOIC-8_L4.9-W3.9-P1.27-LS6.0-BL, symbol Amplifier_Operational:NE5532
- added C17: 10uF, symbol Device:C_Polarized
- added C18, C20, C22: 220uF, symbol Device:C_Polarized
- added C19, C21, C23: 100nF, symbol Device:C
- added Q1: BC549, Package_TO_SOT_THT:TO-92_Inline, symbol Transistor_BJT:BC549
- added R19: 10k, symbol Device:R
- added SW1: SW_DPST, symbol Switch:SW_DPST
- added U1: NMA1209DC, Converter_DCDC:Converter_DCDC_Murata_NMAxxxxDC_THT, symbol Regulator_Switching:NMA1209DC
- added U4: NE5532DR, PCM_JLCPCB:SOIC-8_L4.9-W3.9-P1.27-LS6.0-BL, symbol PCM_JLCPCB-Analog:Op-Amp, NE5532DR
- C9: value 33uF -> 33uF -> 10uF
- R16: value 5.1K -> 2.2K
Connections:
- net +9V: now also C20.1, C21.1, SW1.4, U1.9 (VOUT+), U4.8 (VCC)
- net -9V: now also C22.2, C23.2, U1.11 (VOUT-), U4.4 (GND)
- net GND: now also C17.2, C18.2, C19.2, C20.2, C21.2, C22.1, C23.1, Q1.3 (E), U1.1 (VIN-), U1.8 (0V)
- net at R10.2: now also U4.3 (IN1+)
- net at C10.2, R17.2, R20.2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: now also U4.1 (OUT1)
- net at C10.1, R12.2, R16.1: now also U4.2 (IN1-)
- net at Left_Output1.1 (Pin_1), R20.1: now also Q1.1 (C)
- new net: C17.1, Q1.2 (B), R19.1
- new net: R19.2, SW1.3
- new net +5V: C18.1, C19.1, U1.14 (VIN+)
- no-connect marks 1 -> 3
Other:
- note added: "Adjustable gain: 1 + (R16 + RV2)/R12 = 4.2 - 77.76 Gain"
- note added: "C10 High-freq / treble cutoff Increase -> Remove high pitch Decrease -> Allow more high pitch"
- note added: "C8 Low-freq / bass cutoff Increase -> More bass Decrease -> Remove more bass"
- note added: "C9 Low-freq / bass cutoff Increase -> More bass Decrease -> Remove more bass Similar to C8 but less important?"
- note added: "Left Channel (Replicate for right channel)"
- note added: "Mute circuit / switch"
- note added: "RC 10uF -> 100ms 4.7uF -> 47ms"
- note removed: "Add decoupling capacitor to V+ and V-"
- note removed: "C8 Low-freq / bass cutoff Increase -> More bass Decrease -> Remove more bass C10 High-freq / treble cutoff Increase -> Remove high pitch Decrease -> Allow more high pitch"
- moved on the sheet: C10, C8, C9, Left_3, Left_Output1, R10, R12, R14, R16, R17, R20, R8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
